Commit message: expand joint range

File: mani_skill/assets/robots/RJ2506/urdf/RJ2506_leftarm_panda_hand.urdf (robot description, URDF)
Before this commit: robot RJ2506, 26 links, 25 joints
Joints:
- joint body_joint1: limit lower=-1.57 upper=1.57 effort=0 velocity=0 -> lower=-3.14 upper=3.14 effort=0 velocity=0
- joint body_joint2: limit lower=0 upper=0.75 effort=0 velocity=0 -> lower=-3.14 upper=3.14 effort=0 velocity=0
- joint left_arm_joint3: limit lower=0 upper=1.57 effort=0 velocity=0 -> lower=-3.14 upper=3.14 effort=0 velocity=0
