Commit message: add back cam to rj2506 left hand

File: mani_skill/assets/robots/RJ2506/urdf/RJ2506_leftarm_only_noagv.urdf (robot description, URDF)
Before this commit: robot RJ2506, 24 links, 23 joints
Links:
- added link left_hand_back_cam, mass 0.0958667621444379; collision box size=0.0215 0.041 0.041; visual box size=0.0215 0.041 0.041
Joints:
- added joint left_hand_back_cam_joint: type fixed, parent left_hand_base, child left_hand_back_cam, origin xyz=0.09990000000000057 0 0.129655988461576 rpy=3.1415926 -2.094395102 0, axis 0 0 0

Commit message: update rj2506 moxing

File: mani_skill/assets/robots/RJ2506/urdf/RJ2506_leftarm_only_noagv.urdf (robot description, URDF)
Before this commit: robot RJ2506, 25 links, 24 joints
Joints:
- joint body_joint2: limit lower=-3.14 upper=3.14 effort=0 velocity=0 -> lower=0 upper=3.14 effort=0 velocity=0

Commit message: rj2506 ppo PickCube-v1 done

File: mani_skill/assets/robots/RJ2506/urdf/RJ2506_leftarm_only_noagv.urdf (robot description, URDF)
Before this commit: robot RJ2506, 25 links, 24 joints
Links:
- link left_hand_tcp: geometry 
Joints:
- joint body_joint2: limit lower=0 upper=3.14 effort=0 velocity=0 -> lower=-3.14 upper=3.14 effort=0 velocity=0
